Commit message: Original URDF file before modification

File: ROS/turtlebot3/turtlebot3_description/urdf/turtlebot3_burger.urdf.xacro (robot description, xacro)
@@ -34,5 +34,5 @@
     <parent link="base_link"/>
     <child link="wheel_left_link"/>
-    <origin xyz="0.035 0.08 0.023" rpy="${-M_PI*0.5} 0 0"/> <!-- origin xyz="0.115 0.08 0.023" -->
+    <origin xyz="0.0 0.08 0.023" rpy="${-M_PI*0.5} 0 0"/>
     <axis xyz="0 0 1"/>
   </joint>
@@ -62,5 +62,5 @@
     <parent link="base_link"/>
     <child link="wheel_right_link"/>
-    <origin xyz="0.035 -0.08 0.023" rpy="${-M_PI*0.5} 0 0"/> <!-- origin xyz="0.115 -0.08 0.023" -->
+    <origin xyz="0.0 -0.08 0.023" rpy="${-M_PI*0.5} 0 0"/>
     <axis xyz="0 0 1"/>
   </joint>
@@ -87,62 +87,4 @@
     </inertial>
   </link>
-<!-- Added in lines below-->
-  <joint name="wheel_left_joint_rear" type="continuous">
-    <parent link="base_link"/>
-    <child link="wheel_left_link_rear"/>
-    <origin xyz="-0.128 0.08 0.023" rpy="${-M_PI*0.5} 0 0"/>  <!-- short monster: <origin xyz="-0.035 0.08 0.023" rpy="${-M_PI*0.5} 0 0"/>, orig monster: origin xyz="-0.115 0.08 0.023" -->
-    <axis xyz="0 0 1"/>
-  </joint>
-  <link name="wheel_left_link_rear">
-    <visual>
-      <origin xyz="0 0 0" rpy="${M_PI*0.5} 0 0"/>
-      <geometry>
-        <mesh filename="package://turtlebot3_description/meshes/wheels/left_tire.stl" scale="0.001 0.001 0.001"/>
-      </geometry>
-      <material name="dark"/>
-    </visual>
-    <collision>
-      <origin xyz="0 0 0" rpy="0 0 0"/>
-      <geometry>
-        <cylinder length="0.018" radius="0.033"/>
-      </geometry>
-    </collision>
-    <inertial>
-      <origin xyz="0 0 0" />
-      <mass value="0.01" />
-      <inertia ixx="0.001" ixy="0.0" ixz="0.0"
-               iyy="0.001" iyz="0.0"
-               izz="0.001" />
-    </inertial>
-  </link>
-  <joint name="wheel_right_joint_rear" type="continuous">
-    <parent link="base_link"/>
-    <child link="wheel_right_link_rear"/>
-    <origin xyz="-0.128 -0.08 0.023" rpy="${-M_PI*0.5} 0 0"/> <!-- <origin xyz="-0.035 -0.08 0.023" rpy="${-M_PI*0.5} 0 0"/> , Orig Monster: 0.035 origin xyz="-0.115 -0.08 0.023" -->
-    <axis xyz="0 0 1"/>
-  </joint>
-  <link name="wheel_right_link_rear">
-    <visual>
-      <origin xyz="0 0 0" rpy="${M_PI*0.5} 0 0"/>
-      <geometry>
-        <mesh filename="package://turtlebot3_description/meshes/wheels/right_tire.stl" scale="0.001 0.001 0.001"/>
-      </geometry>
-      <material name="dark"/>
-    </visual>
-    <collision>
-      <origin xyz="0 0 0" rpy="0 0 0"/>
-      <geometry>
-        <cylinder length="0.018" radius="0.033"/>
-      </geometry>
-    </collision>
-    <inertial>
-      <origin xyz="0 0 0" />
-      <mass value="0.01" />
-      <inertia ixx="0.001" ixy="0.0" ixz="0.0"
-               iyy="0.001" iyz="0.0"
-               izz="0.001" />
-    </inertial>
-  </link>
-<!-- Added in lines above-->
   <joint name="caster_back_joint" type="fixed">
     <parent link="base_link"/>

Commit message: Modified robot description file, URDF to include rear wheels

File: ROS/turtlebot3/turtlebot3_description/urdf/turtlebot3_burger.urdf.xacro (robot description, xacro)
@@ -34,5 +34,5 @@
     <parent link="base_link"/>
     <child link="wheel_left_link"/>
-    <origin xyz="0.0 0.08 0.023" rpy="${-M_PI*0.5} 0 0"/>
+    <origin xyz="0.035 0.08 0.023" rpy="${-M_PI*0.5} 0 0"/> <!-- origin xyz="0.115 0.08 0.023" -->
     <axis xyz="0 0 1"/>
   </joint>
@@ -62,5 +62,5 @@
     <parent link="base_link"/>
     <child link="wheel_right_link"/>
-    <origin xyz="0.0 -0.08 0.023" rpy="${-M_PI*0.5} 0 0"/>
+    <origin xyz="0.035 -0.08 0.023" rpy="${-M_PI*0.5} 0 0"/> <!-- origin xyz="0.115 -0.08 0.023" -->
     <axis xyz="0 0 1"/>
   </joint>
@@ -87,4 +87,62 @@
     </inertial>
   </link>
+<!-- Added in lines below-->
+  <joint name="wheel_left_joint_rear" type="continuous">
+    <parent link="base_link"/>
+    <child link="wheel_left_link_rear"/>
+    <origin xyz="-0.128 0.08 0.023" rpy="${-M_PI*0.5} 0 0"/>  <!-- short monster: <origin xyz="-0.035 0.08 0.023" rpy="${-M_PI*0.5} 0 0"/>, orig monster: origin xyz="-0.115 0.08 0.023" -->
+    <axis xyz="0 0 1"/>
+  </joint>
+  <link name="wheel_left_link_rear">
+    <visual>
+      <origin xyz="0 0 0" rpy="${M_PI*0.5} 0 0"/>
+      <geometry>
+        <mesh filename="package://turtlebot3_description/meshes/wheels/left_tire.stl" scale="0.001 0.001 0.001"/>
+      </geometry>
+      <material name="dark"/>
+    </visual>
+    <collision>
+      <origin xyz="0 0 0" rpy="0 0 0"/>
+      <geometry>
+        <cylinder length="0.018" radius="0.033"/>
+      </geometry>
+    </collision>
+    <inertial>
+      <origin xyz="0 0 0" />
+      <mass value="0.01" />
+      <inertia ixx="0.001" ixy="0.0" ixz="0.0"
+               iyy="0.001" iyz="0.0"
+               izz="0.001" />
+    </inertial>
+  </link>
+  <joint name="wheel_right_joint_rear" type="continuous">
+    <parent link="base_link"/>
+    <child link="wheel_right_link_rear"/>
+    <origin xyz="-0.128 -0.08 0.023" rpy="${-M_PI*0.5} 0 0"/> <!-- <origin xyz="-0.035 -0.08 0.023" rpy="${-M_PI*0.5} 0 0"/> , Orig Monster: 0.035 origin xyz="-0.115 -0.08 0.023" -->
+    <axis xyz="0 0 1"/>
+  </joint>
+  <link name="wheel_right_link_rear">
+    <visual>
+      <origin xyz="0 0 0" rpy="${M_PI*0.5} 0 0"/>
+      <geometry>
+        <mesh filename="package://turtlebot3_description/meshes/wheels/right_tire.stl" scale="0.001 0.001 0.001"/>
+      </geometry>
+      <material name="dark"/>
+    </visual>
+    <collision>
+      <origin xyz="0 0 0" rpy="0 0 0"/>
+      <geometry>
+        <cylinder length="0.018" radius="0.033"/>
+      </geometry>
+    </collision>
+    <inertial>
+      <origin xyz="0 0 0" />
+      <mass value="0.01" />
+      <inertia ixx="0.001" ixy="0.0" ixz="0.0"
+               iyy="0.001" iyz="0.0"
+               izz="0.001" />
+    </inertial>
+  </link>
+<!-- Added in lines above-->
   <joint name="caster_back_joint" type="fixed">
     <parent link="base_link"/>
